File: Micro.sch (KiCad schematic (older format))
At the start: 26 parts, among them J1 USB_B_Mini, J2 Programmer, J3 Conn_01x13, J4 Conn_01x13, J5 Conn_01x13, U1 ADP2108AUJ-3.3, U2 MK20DX256VLH7, Y1 16 Mhz

Commit message: Cleaned up and set footprints
Parts:
- C1, C10, C3, C4, C5, C6, C7, C8, C9, FB1, FB2: footprint (none) -> Capacitor_SMD:C_0805_2012Metric_Pad1.15x1.40mm_HandSolder
- C2: footprint (none) -> Capacitor_SMD:CP_Elec_5x3.9
- J2: footprint (none) -> Connector_PinHeader_2.00mm:PinHeader_2x04_P2.00mm_Vertical
- J3, J4, J5: footprint (none) -> Connector_PinHeader_2.54mm:PinHeader_1x13_P2.54mm_Vertical
- L1: footprint (none) -> Inductor_SMD:L_0805_2012Metric_Pad1.15x1.40mm_HandSolder
- R1, R2, R3: footprint (none) -> Resistor_SMD:R_0805_2012Metric_Pad1.15x1.40mm_HandSolder
- TP1, TP2: footprint (none) -> TestPoint:TestPoint_Loop_D2.54mm_Drill1.5mm_Beaded
- Y1: footprint (none) -> Crystal:Crystal_HC49-U_Vertical
Connections:
- wire segments 136 -> 132
Changed lines of the file:
@@
 EESchema Schematic File Version 4
+LIBS:Micro-cache
 EELAYER 29 0
 EELAYER END
@@
 F 0 "J2" H 1400 3767 50  0000 C CNN
 F 1 "Programmer" H 1400 3676 50  0000 C CNN
-F 2 "" H 1350 3450 50  0001 C CNN
+F 2 "Connector_PinHeader_2.00mm:PinHeader_2x04_P2.00mm_Vertical" H 1350 3450 50  0001 C CNN
 F 3 "~" H 1350 3450 50  0001 C CNN
 	1    1350 3450
@@
 F 0 "R1" V 1345 1450 50  0000 C CNN
 F 1 "33" V 1436 1450 50  0000 C CNN
-F 2 "" V 1590 1440 50  0001 C CNN
+F 2 "Resistor_SMD:R_0805_2012Metric_Pad1.15x1.40mm_HandSolder" V 1590 1440 50  0001 C CNN
 F 3 "~" H 1550 1450 50  0001 C CNN
 	1    1550 1450
@@
 F 0 "R2" V 1345 1550 50  0000 C CNN
 F 1 "33" V 1436 1550 50  0000 C CNN
-F 2 "" V 1590 1540 50  0001 C CNN
+F 2 "Resistor_SMD:R_0805_2012Metric_Pad1.15x1.40mm_HandSolder" V 1590 1540 50  0001 C CNN
 F 3 "~" H 1550 1550 50  0001 C CNN
 	1    1550 1550
@@
 Wire Wire Line
 	1300 1550 1400 1550
-Text Label 1900 1650 2    50   ~ 0
-PTA1
 Wire Wire Line
 	1700 1450 1900 1450
@@
 Text Label 1900 1550 2    50   ~ 0
 USBM
-Wire Wire Line
-	1300 1650 1900 1650
 $Comp
 L Regulator_Switching:ADP2108AUJ-3.3 U1
@@
 F 0 "C1" H 2265 1446 50  0000 L CNN
 F 1 "4.7uF" H 2265 1355 50  0000 L CNN
-F 2 "" H 2188 1250 50  0001 C CNN
+F 2 "Capacitor_SMD:C_0805_2012Metric_Pad1.15x1.40mm_HandSolder" H 2188 1250 50  0001 C CNN
 F 3 "~" H 2150 1400 50  0001 C CNN
 	1    2150 1400
@@
 F 0 "L1" H 3350 1465 50  0000 C CNN
 F 1 "1uH" H 3350 1374 50  0000 C CNN
-F 2 "" H 3350 1250 50  0001 C CNN
+F 2 "Inductor_SMD:L_0805_2012Metric_Pad1.15x1.40mm_HandSolder" H 3350 1250 50  0001 C CNN
 F 3 "~" H 3350 1250 50  0001 C CNN
 	1    3350 1250
@@
 F 0 "C2" H 3715 1646 50  0000 L CNN
 F 1 "10uF" H 3715 1555 50  0000 L CNN
-F 2 "" H 3638 1450 50  0001 C CNN
+F 2 "Capacitor_SMD:CP_Elec_5x3.9" H 3638 1450 50  0001 C CNN
 F 3 "~" H 3600 1600 50  0001 C CNN
 	1    3600 1600
@@
 F 0 "C6" H 6415 1446 50  0000 L CNN
 F 1 "2.2uF" H 6415 1355 50  0000 L CNN
-F 2 "" H 6338 1250 50  0001 C CNN
+F 2 "Capacitor_SMD:C_0805_2012Metric_Pad1.15x1.40mm_HandSolder" H 6338 1250 50  0001 C CNN
 F 3 "~" H 6300 1400 50  0001 C CNN
 	1    6300 1400
@@
 F 0 "C5" H 6015 1446 50  0000 L CNN
 F 1 "0.1uF" H 6015 1355 50  0000 L CNN
-F 2 "" H 5938 1250 50  0001 C CNN
+F 2 "Capacitor_SMD:C_0805_2012Metric_Pad1.15x1.40mm_HandSolder" H 5938 1250 50  0001 C CNN
 F 3 "~" H 5900 1400 50  0001 C CNN
 	1    5900 1400
@@
 F 0 "C4" H 5615 1446 50  0000 L CNN
 F 1 "0.1uF" H 5615 1355 50  0000 L CNN
-F 2 "" H 5538 1250 50  0001 C CNN
+F 2 "Capacitor_SMD:C_0805_2012Metric_Pad1.15x1.40mm_HandSolder" H 5538 1250 50  0001 C CNN
 F 3 "~" H 5500 1400 50  0001 C CNN
 	1    5500 1400
@@
 F 0 "C3" H 5215 1446 50  0000 L CNN
 F 1 "0.1uF" H 5215 1355 50  0000 L CNN
-F 2 "" H 5138 1250 50  0001 C CNN
+F 2 "Capacitor_SMD:C_0805_2012Metric_Pad1.15x1.40mm_HandSolder" H 5138 1250 50  0001 C CNN
 F 3 "~" H 5100 1400 50  0001 C CNN
 	1    5100 1400
@@
 F 0 "Y1" V 6004 3119 50  0000 R CNN
 F 1 "16 Mhz" V 6095 3119 50  0000 R CNN
-F 2 "" H 6050 3250 50  0001 C CNN
+F 2 "Crystal:Crystal_HC49-U_Vertical" H 6050 3250 50  0001 C CNN
 F 3 "~" H 6050 3250 50  0001 C CNN
 	1    6050 3250
@@
 F 0 "TP2" H 4158 1368 50  0000 L CNN
 F 1 "TestPoint" H 4158 1277 50  0000 L CNN
-F 2 "" H 4300 1250 50  0001 C CNN
+F 2 "TestPoint:TestPoint_Loop_D2.54mm_Drill1.5mm_Beaded" H 4300 1250 50  0001 C CNN
 F 3 "~" H 4300 1250 50  0001 C CNN
 	1    4100 1250
@@
 F 0 "TP1" H 1258 2118 50  0000 L CNN
 F 1 "TestPoint" H 1258 2027 50  0000 L CNN
-F 2 "" H 1400 2000 50  0001 C CNN
+F 2 "TestPoint:TestPoint_Loop_D2.54mm_Drill1.5mm_Beaded" H 1400 2000 50  0001 C CNN
 F 3 "~" H 1400 2000 50  0001 C CNN
 	1    1200 2000
@@
 F 0 "J4" H 9750 2850 50  0000 C CNN
 F 1 "Conn_01x13" H 9750 2950 50  0000 C CNN
-F 2 "" H 9450 2950 50  0001 C CNN
+F 2 "Connector_PinHeader_2.54mm:PinHeader_1x13_P2.54mm_Vertical" H 9450 2950 50  0001 C CNN
 F 3 "~" H 9450 2950 50  0001 C CNN
 	1    9450 2950
@@
 F 0 "J3" H 9750 1450 50  0000 C CNN
 F 1 "Conn_01x13" H 9750 1550 50  0000 C CNN
-F 2 "" H 9450 1550 50  0001 C CNN
+F 2 "Connector_PinHeader_2.54mm:PinHeader_1x13_P2.54mm_Vertical" H 9450 1550 50  0001 C CNN
 F 3 "~" H 9450 1550 50  0001 C CNN
 	1    9450 1550
@@
 L power:GND #PWR0111
 U 1 1 5D41B7C6
-P 8950 950
-F 0 "#PWR0111" H 8950 700 50  0001 C CNN
-F 1 "GND" H 8955 777 50  0000 C CNN
-F 2 "" H 8950 950 50  0001 C CNN
-F 3 "" H 8950 950 50  0001 C CNN
-	1    8950 950
-	1    0    0    -1
-$EndComp
-Wire Wire Line
-	8950 950  9100 950
-Wire Wire Line
-	9100 950  9100 1050
-Wire Wire Line
-	9100 1050 9250 1050
+P 9200 5150
+F 0 "#PWR0111" H 9200 4900 50  0001 C CNN
+F 1 "GND" H 9205 4977 50  0000 C CNN
+F 2 "" H 9200 5150 50  0001 C CNN
+F 3 "" H 9200 5150 50  0001 C CNN
+	1    9200 5150
+	1    0    0    -1
+$EndComp
 $Comp
 L power:+3.3V #PWR0112
 U 1 1 5D420696
-P 8950 900
-F 0 "#PWR0112" H 8950 750 50  0001 C CNN
-F 1 "+3.3V" H 8965 1073 50  0000 C CNN
-F 2 "" H 8950 900 50  0001 C CNN
-F 3 "" H 8950 900 50  0001 C CNN
-	1    8950 900
-	1    0    0    -1
-$EndComp
-Wire Wire Line
-	8950 900  9150 900
-Wire Wire Line
-	9150 900  9150 950
-Wire Wire Line
-	9150 950  9250 950
+P 9200 950
+F 0 "#PWR0112" H 9200 800 50  0001 C CNN
+F 1 "+3.3V" H 9215 1123 50  0000 C CNN
+F 2 "" H 9200 950 50  0001 C CNN
+F 3 "" H 9200 950 50  0001 C CNN
+	1    9200 950
+	1    0    0    -1
+$EndComp
 $Comp
 L Connector_Generic:Conn_01x13 J5
@@
 F 0 "J5" H 9750 4350 50  0000 C CNN
 F 1 "Conn_01x13" H 9750 4450 50  0000 C CNN
-F 2 "" H 9450 4450 50  0001 C CNN
+F 2 "Connector_PinHeader_2.54mm:PinHeader_1x13_P2.54mm_Vertical" H 9450 4450 50  0001 C CNN
 F 3 "~" H 9450 4450 50  0001 C CNN
 	1    9450 4450
@@
 F 0 "C9" H 6415 2446 50  0000 L CNN
 F 1 "0.1uF" H 6415 2355 50  0000 L CNN
-F 2 "" H 6338 2250 50  0001 C CNN
+F 2 "Capacitor_SMD:C_0805_2012Metric_Pad1.15x1.40mm_HandSolder" H 6338 2250 50  0001 C CNN
 F 3 "~" H 6300 2400 50  0001 C CNN
 	1    6300 2400
@@
 F 0 "FB1" V 4750 2550 50  0000 C CNN
 F 1 "Ferrite" V 4650 2550 50  0000 C CNN
-F 2 "" V 4830 2550 50  0001 C CNN
+F 2 "Capacitor_SMD:C_0805_2012Metric_Pad1.15x1.40mm_HandSolder" V 4830 2550 50  0001 C CNN
 F 3 "~" H 4900 2550 50  0001 C CNN
 	1    4900 2550
@@
 F 0 "C7" H 5215 2446 50  0000 L CNN
 F 1 "2.2uF" H 5215 2355 50  0000 L CNN
-F 2 "" H 5138 2250 50  0001 C CNN
+F 2 "Capacitor_SMD:C_0805_2012Metric_Pad1.15x1.40mm_HandSolder" H 5138 2250 50  0001 C CNN
 F 3 "~" H 5100 2400 50  0001 C CNN
 	1    5100 2400
@@
 F 0 "FB2" H 4750 2100 50  0000 L CNN
 F 1 "Ferrite" H 4700 2000 50  0000 L CNN
-F 2 "" V 5030 2050 50  0001 C CNN
+F 2 "Capacitor_SMD:C_0805_2012Metric_Pad1.15x1.40mm_HandSolder" V 5030 2050 50  0001 C CNN
 F 3 "~" H 5100 2050 50  0001 C CNN
 	1    5100 2050
@@
 F 0 "R3" V 5445 2250 50  0000 C CNN
 F 1 "470" V 5536 2250 50  0000 C CNN
-F 2 "" V 5690 2240 50  0001 C CNN
+F 2 "Resistor_SMD:R_0805_2012Metric_Pad1.15x1.40mm_HandSolder" V 5690 2240 50  0001 C CNN
 F 3 "~" H 5650 2250 50  0001 C CNN
 	1    5650 2250
@@
 F 0 "C8" H 5965 2446 50  0000 L CNN
 F 1 "0.1uF" H 5965 2355 50  0000 L CNN
-F 2 "" H 5888 2250 50  0001 C CNN
+F 2 "Capacitor_SMD:C_0805_2012Metric_Pad1.15x1.40mm_HandSolder" H 5888 2250 50  0001 C CNN
 F 3 "~" H 5850 2400 50  0001 C CNN
 	1    5850 2400
@@
 F 0 "C10" H 5265 3946 50  0000 L CNN
 F 1 "0.1uF" H 5265 3855 50  0000 L CNN
-F 2 "" H 5188 3750 50  0001 C CNN
+F 2 "Capacitor_SMD:C_0805_2012Metric_Pad1.15x1.40mm_HandSolder" H 5188 3750 50  0001 C CNN
 F 3 "~" H 5150 3900 50  0001 C CNN
 	1    5150 3900
@@
 	5150 3750 6800 3750
 Connection ~ 5150 3750
+Wire Wire Line
+	9250 1050 9200 1050
+Wire Wire Line
+	9200 1050 9200 5150
+Wire Wire Line
+	9200 950  9250 950
 $EndSCHEMATC
