File: Micro.kicad_pcb (KiCad board)
At the start: 2 copper layers, 26 parts, among them J1 USB_B_Mini, J2 Programmer, J3 Conn_01x13, J4 Conn_01x13, J5 Conn_01x13, U1 ADP2108AUJ-3.3, U2 MK20DX256VLH7, Y1 16 Mhz

Commit message: Continued routing
Parts:
- moved TP2 48.1 mm to (127.9, 87.2)
- moved FB1 46.0 mm to (136.1, 103.6), turned to 90 degrees
- moved TP1 44.0 mm to (125.7, 99.8)
- moved J5 43.4 mm to (132.0, 117.0)
- moved C10 36.6 mm to (141.6, 108.4), turned to 270 degrees
- moved R3 36.0 mm to (139.4, 99.8), turned to 90 degrees
- moved J3 32.3 mm to (169.4, 112.0), turned to 180 degrees
- moved C5 17.5 mm to (162.3, 109.7)
- moved J2 17.4 mm to (150.7, 108.1), turned to 270 degrees
- moved C3 7.35 mm to (156.5, 110.2)
- moved FB2 5.11 mm to (135.2, 96.9)
- moved C7 4.30 mm to (136.1, 99.8)
- moved C8 3.93 mm to (132.8, 99.8), turned to 270 degrees
- moved C4 3.53 mm to (154.8, 90.7), turned to 0 degrees
- moved J4 1.49 mm to (131.7, 80.0)
Routing:
- net +3V3: track 22.5 -> 35.6 mm
- net GND: track 6.05 -> 18.9 mm
- net /RST: track 0.00 -> 10.1 mm, vias 0 -> 1
- net Net-(C7-Pad1): track 0.00 -> 7.94 mm
- net /PTA3: track 17.6 -> 10.5 mm
- net /PTA2: track 15.8 -> 8.79 mm
- net Net-(C8-Pad1): track 4.68 -> 10.5 mm
- net /PTA1: track 12.1 -> 8.53 mm
- net /PTA0: track 8.85 -> 8.27 mm
- net Net-(C7-Pad2): track 11.9 -> 12.4 mm, vias 2 -> 0
